File: ArcadeEncoder.kicad_pcb (KiCad board)
At the start: 2 copper layers, 56.6 x 38.7 mm, 8 parts, among them J1 DB15_Male, J2 DB9_Male, U1 ProMicro

Commit message: Updated to KiCad 6
Parts:
- J1: footprint halibs:D-Sub_Connector_15P-Male -> haus-automatisierung:D-Sub_Connector_15P-Male
- J2: footprint halibs:D-Sub_Connector_9P-Male -> haus-automatisierung:D-Sub_Connector_9P-Male
- U1: footprint halibs:ArduinoProMicro -> haus-automatisierung:ArduinoProMicro
Connections:
- J1 pad 9: Net-(J1-Pad9) -> unconnected-(J1-Pad9)
- U1 pad 10: Net-(U1-Pad10) -> unconnected-(U1-Pad10)
- U1 pad 11: Net-(U1-Pad11) -> unconnected-(U1-Pad11)
- U1 pad 12: Net-(U1-Pad12) -> unconnected-(U1-Pad12)
- U1 pad 13: Net-(U1-Pad13) -> unconnected-(U1-Pad13)
- U1 pad 22: Net-(U1-Pad22) -> unconnected-(U1-Pad22)
- U1 pad 24: Net-(U1-Pad24) -> unconnected-(U1-Pad24)
- U1 pad 8: Net-(U1-Pad8) -> unconnected-(U1-Pad8)
- U1 pad 9: Net-(U1-Pad9) -> unconnected-(U1-Pad9)
Routing:
- net +5V: track 58.6 -> 57.5 mm
Other:
- net class Default removed
